File: beagledancer.kicad_pcb (KiCad board)
At the start: 2 copper layers, 32 x 23.1 mm, 12 parts, among them J1 USB-MICRO-B, P9 BeagleBone, U1 MAX3421, X1 XTAL4PIN

Commit message: Add labels to silkscreen
Parts:
- moved C3 0.92 mm to (213.6, 155.2), turned to 180 degrees
Changed lines of the file:
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@@
     (links 32)
     (no_connects 0)
-    (area 198.323999 136.601999 230.428001 159.816001)
+    (area 191.001227 135.0518 230.428001 160.708622)
     (thickness 1.6)
     (drawings 10)
@@
   )
   (module SM0603_Capa (layer F.Cu)
-    (at 214.122 155.956 270)
+    (at 213.614 155.194 180)
     (attr smd)
-    (fp_text reference C3 (at 0 0 360) (layer F.SilkS)
-      (effects (font (size 0.508 0.4572) (thickness 0.1143)))
-    )
-    (fp_text value 18pf (at -1.651 0 360) (layer F.SilkS)
+    (fp_text reference C3 (at 0 0 270) (layer F.SilkS)
+      (effects (font (size 0.508 0.4572) (thickness 0.1143)))
+    )
+    (fp_text value 18pf (at -1.651 0 270) (layer F.SilkS)
       (effects (font (size 0.508 0.4572) (thickness 0.1143)))
     )
@@
     (fp_line (start 1.19888 -0.635) (end 1.19888 0.635) (layer F.SilkS) (width 0.11938))
     (fp_line (start -1.19888 0.635) (end -1.19888 -0.635) (layer F.SilkS) (width 0.11938))
-    (pad 1 smd rect (at -0.762 0 270) (size 0.635 1.143)
+    (pad 1 smd rect (at -0.762 0 180) (size 0.635 1.143)
       (layers F.Cu F.Paste F.Mask)
       (net 7 /XI)
     )
-    (pad 2 smd rect (at 0.762 0 270) (size 0.635 1.143)
+    (pad 2 smd rect (at 0.762 0 180) (size 0.635 1.143)
       (layers F.Cu F.Paste F.Mask)
       (net 9 GND)
@@
   (module GSG-USB-MICROB-FCI-10103594 (layer F.Cu)
     (at 198.1708 152.0952)
-    (fp_text reference J1 (at 2.49936 0) (layer F.SilkS)
+    (fp_text reference J1 (at 2.49936 0) (layer F.SilkS) hide
       (effects (font (thickness 0.3048)))
     )
@@
     (descr "Connecteurs 2 pins")
     (tags "CONN DEV")
-    (fp_text reference JP1 (at 0 -1.905 180) (layer F.SilkS)
+    (fp_text reference JP1 (at 0 -1.905 180) (layer F.SilkS) hide
       (effects (font (size 0.762 0.762) (thickness 0.1524)))
     )
@@
   (module GSG-XTAL3.2x2.5mm (layer F.Cu)
     (at 217.424 155.956 270)
-    (fp_text reference X1 (at 0 0 270) (layer F.SilkS)
+    (fp_text reference X1 (at 0 0 270) (layer F.SilkS) hide
       (effects (font (size 1.00076 1.00076) (thickness 0.2032)))
     )
@@
   (module MAX3421 (layer F.Cu)
     (at 222.25 150.622 90)
-    (fp_text reference U1 (at 0.1 0.725 90) (layer F.SilkS)
+    (fp_text reference U1 (at 0.1 0.725 90) (layer F.SilkS) hide
       (effects (font (size 0.75 0.75) (thickness 0.075)))
     )
@@
   (segment (start 220.4875 156.9565) (end 220.4875 153.8595) (width 0.2032) (layer F.Cu) (net 8) (status 30))
   (segment (start 220.38818 157.05582) (end 220.4875 156.9565) (width 0.2032) (layer F.Cu) (net 8) (status 30))
-  (segment (start 225.41 151.372) (end 224.143 151.372) (width 0.254) (layer F.Cu) (net 9) (status 400000))
+  (segment (start 212.852 155.194) (end 211.455 155.194) (width 0.254) (layer F.Cu) (net 9) (status 400000))
+  (via (at 211.455 155.194) (size 1.016) (layers F.Cu B.Cu) (net 9))
+  (segment (start 225.41 151.372) (end 224.143 151.372) (width 0.254) (layer F.Cu) (net 9))
   (via (at 223.647 150.876) (size 1.016) (layers F.Cu B.Cu) (net 9))
   (segment (start 224.143 151.372) (end 223.647 150.876) (width 0.254) (layer F.Cu) (net 9))
-  (segment (start 219.09 149.872) (end 220.103 149.872) (width 0.254) (layer F.Cu) (net 9) (status 400000))
+  (segment (start 219.09 149.872) (end 220.103 149.872) (width 0.254) (layer F.Cu) (net 9))
   (via (at 220.853 150.622) (size 1.016) (layers F.Cu B.Cu) (net 9))
   (segment (start 220.103 149.872) (end 220.853 150.622) (width 0.254) (layer F.Cu) (net 9))
@@
   (via (at 204.978 148.59) (size 1.016) (layers F.Cu B.Cu) (net 9))
   (segment (start 205.0542 148.5138) (end 204.978 148.59) (width 0.254) (layer F.Cu) (net 9))
-  (segment (start 214.122 156.718) (end 212.598 156.718) (width 0.254) (layer F.Cu) (net 9))
-  (via (at 212.598 156.718) (size 1.016) (layers F.Cu B.Cu) (net 9))
   (segment (start 221.996 156.972) (end 223.266 156.972) (width 0.254) (layer F.Cu) (net 9))
   (via (at 223.266 156.972) (size 1.016) (layers F.Cu B.Cu) (net 9))
